File: opto-comp.kicad_pcb (KiCad board)
At the start: 2 copper layers, 57 x 94 mm, 99 parts, among them J1 CALIB_A, J2 INPUT_JACK, J3 OUTPUT_JACK, J4 POWER_CONN, J5 BYPASS_NOISE_FILTER, J6 CALIB_B, Q1 2SC1815, Q2 2SC1815, Q3 2SC1815, SW1 SW_DPDT_x2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

Commit message: fix LCR pattern, add credit
Parts:
- U6, U7: moved to F.Cu
- moved U7 5.63 mm to (105.2, 108.0)
- moved U6 4.48 mm to (75.9, 103.0)
Routing:
- net CDS_B: track 42.7 -> 38.2 mm
- net CDS_A: track 30.5 -> 34.4 mm
- net Net-(D9-Pad1): track 14.1 -> 16.1 mm
- net Vbias: track 135.5 -> 137.5 mm
- net Net-(U6-Pad1): track 28.3 -> 29.8 mm
- net Net-(D1-Pad2): track 35.2 -> 34.1 mm
Other:
- board text added: "MST Compress v1.0.1"
- board text added: "https://meso.tokyo/"

Commit message: Replace LM324 to NJM2902N
Parts:
- U5: value LM324 -> NJM2902N
Changed lines of the file:
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@@
       (effects (font (size 1 1) (thickness 0.15)) (justify mirror))
     )
-    (fp_text value "LM324" (at 3.81 -17.57) (layer "B.Fab")
+    (fp_text value "NJM2902N" (at 3.81 -17.57) (layer "B.Fab")
       (effects (font (size 1 1) (thickness 0.15)) (justify mirror))
     )
